Commit message: Renamed links of pepito robot, and created new publisher to obtain its position from /map.

File: robots/pepito_robot/pepito_description/urdf/pepito_arm-up_no-head.urdf (robot description, URDF)
Before this commit: robot pepito, 13 links, 12 joints
Links:
- removed link jido_base_footprint
- removed link jido_base_laser_link
- removed link jido_base_link
- added link jido_link_base; visual box size=0.65 0.65 0.40
- added link jido_link_footprint
- added link jido_link_laser
Joints:
- removed joint jido_base_joint
- removed joint jido_laser_joint
- added joint jido_joint_base: type fixed, parent jido_link_footprint, child jido_link_base, origin xyz=0 0 0 rpy=0 0 0
- added joint jido_joint_laser: type fixed, parent jido_link_base, child jido_link_laser, origin xyz=0.37 0 0.3 rpy=0 0 0
- joint pepito_base: parent jido_base_link -> jido_link_base
