Commit message: Updated URDF of pepito robot, now all links and joints are named following convention.

File: robots/pepito_robot/pepito_description/urdf/jido.urdf (robot description, URDF)
Before this commit: robot Jido, 5 links, 4 joints
Links:
- removed link base_footprint
- removed link base_laser_link
- removed link base_link
- removed link head_pan_link
- removed link head_tilt_link
- added link jido_link_base
- added link jido_link_footprint
- added link jido_link_head_pan_
- added link jido_link_head_tilt
- added link jido_link_laser
Joints:
- removed joint base_joint
- removed joint head_pan_joint
- removed joint head_tilt_joint
- removed joint laser_joint
- added joint jido_joint_base: type fixed, parent jido_link_footprint, child jido_link_base, origin xyz=0 0 0 rpy=0 0 0
- added joint jido_joint_head_pan: type continuous, parent jido_link_base, child jido_link_head_pan, origin xyz=0.239 0 1.185 rpy=0 0 0, axis 0 0 1
- added joint jido_joint_head_tilt: type continuous, parent jido_link_head_pan, child jido_link_head_tilt, origin xyz=0 0 0.02 rpy=0 0 0, axis 0 1 0
- added joint jido_joint_laser: type fixed, parent jido_link_base, child jido_link_laser, origin xyz=0.37 0 0.3 rpy=0 0 0

File: robots/pepito_robot/pepito_description/urdf/pepito_config_left.urdf (robot description, URDF)
Before this commit: robot pepito, 15 links, 14 joints
Links:
- removed link jido_base_footprint
- removed link jido_base_laser_link
- removed link jido_base_link
- removed link jido_head_pan_link
- removed link jido_head_tilt_link
- added link jido_link_base; visual box size=0.65 0.65 0.40
- added link jido_link_footprint
- added link jido_link_head_pan_
- added link jido_link_head_tilt
- added link jido_link_laser
Joints:
- removed joint jido_base_joint
- removed joint jido_head_pan_joint
- removed joint jido_head_tilt_joint
- removed joint jido_laser_joint
- added joint jido_joint_base: type fixed, parent jido_link_footprint, child jido_link_base, origin xyz=0 0 0 rpy=0 0 0
- added joint jido_joint_head_pan: type continuous, parent jido_link_base, child jido_link_head_pan, origin xyz=0.239 0 1.185 rpy=0 0 0, axis 0 0 1
- added joint jido_joint_head_tilt: type continuous, parent jido_link_head_pan, child jido_link_head_tilt, origin xyz=0 0 0.02 rpy=0 0 0, axis 0 1 0
- added joint jido_joint_laser: type fixed, parent jido_link_base, child jido_link_laser, origin xyz=0.37 0 0.3 rpy=0 0 0
- joint pepito_base: parent jido_base_link -> jido_link_base

File: robots/pepito_robot/pepito_description/urdf/pepito_config_up.urdf (robot description, URDF)
Before this commit: robot pepito, 15 links, 14 joints
Links:
- removed link jido_base_footprint
- removed link jido_base_laser_link
- removed link jido_base_link
- removed link jido_head_pan_link
- removed link jido_head_tilt_link
- added link jido_link_base; visual box size=0.65 0.65 0.40
- added link jido_link_footprint
- added link jido_link_head_pan_
- added link jido_link_head_tilt
- added link jido_link_laser
Joints:
- removed joint jido_base_joint
- removed joint jido_head_pan_joint
- removed joint jido_head_tilt_joint
- removed joint jido_laser_joint
- added joint jido_joint_base: type fixed, parent jido_link_footprint, child jido_link_base, origin xyz=0 0 0 rpy=0 0 0
- added joint jido_joint_head_pan: type continuous, parent jido_link_base, child jido_link_head_pan, origin xyz=0.239 0 1.185 rpy=0 0 0, axis 0 0 1
- added joint jido_joint_head_tilt: type continuous, parent jido_link_head_pan, child jido_link_head_tilt, origin xyz=0 0 0.02 rpy=0 0 0, axis 0 1 0
- added joint jido_joint_laser: type fixed, parent jido_link_base, child jido_link_laser, origin xyz=0.37 0 0.3 rpy=0 0 0
- joint pepito_base: parent jido_base_link -> jido_link_base
